File: pcb/eurosid.kicad_pcb (KiCad board)
At the start: 2 copper layers, 38 parts, among them J1 Gate 1 In, J10 Stereo jack - MiDI TRS, J11 Conn_01x06_Female, J12 SSD1306_i2c_Oled_Conn_01x04_F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, J13 FRAM_Breakout_i2c_01x08, J14 Audio Out Jack, J2 Gate 2 In, J3 Gate 3 In, J4 Input_Jack_A, J5 Input_Jack_B, J6 Input_Jack_C, J7 Input_Jack_D, J8 Input_Jack_E, J9 Input_Jack_F, SW1 SW_Push_Dual, U2 ATmega1284-PU, U3 PIMORONI_24v_ADC_1_ADS1015IDGS, U5 TL074, U6 PIMORONI_24v_ADC_2_ADS1015IDGS, U7 L78L33_TO92, Y1 Crystal

Commit message: tracked hardware
Parts:
- removed U5: TL074, Package_DIP:DIP-14_W7.62mm_Socket
- removed U6: PIMORONI_24v_ADC_2_ADS1015IDGS, Package_SO:TSSOP-10_3x3mm_P0.5mm
- added ADS1015_breakout_1: ADS1015_breakout, my footprints:ADS1015_breakout, B.Cu at (343.5, 50.2)
- added ADS1015_breakout_2: ADS1015_breakout_2, my footprints:ADS1015_breakout, B.Cu at (343.5, 67.9)
- added C4: 1uf, Capacitor_THT:CP_Radial_D8.0mm_P5.00mm, F.Cu at (102.9, 10.2)
- added C5: 1nf, Capacitor_THT:C_Disc_D8.0mm_W2.5mm_P5.00mm, F.Cu at (126.6, 30.8)
- added C6: CP, Capacitor_THT:CP_Radial_D8.0mm_P2.50mm, F.Cu at (73.9, 10.2)
- added C7: CP, Capacitor_THT:CP_Radial_D8.0mm_P2.50mm, F.Cu at (73.9, 19.7)
- added D10: 1N5817, Diode_THT:D_DO-41_SOD81_P10.16mm_Horizontal, F.Cu at (84.0, 35.1)
- added D7: 1N4148, Diode_THT:D_DO-35_SOD27_P7.62mm_Horizontal, F.Cu at (120.7, 160.7)
- added D8: 1N5817, Diode_THT:D_DO-41_SOD81_P10.16mm_Horizontal, F.Cu at (84.0, 26.6)
- added D9: 1N5817, Diode_THT:D_DO-41_SOD81_P10.16mm_Horizontal, F.Cu at (84.0, 30.9)
- added FDTI_HEADER1: Conn_01x06_Female, Connector_PinSocket_2.54mm:PinSocket_1x06_P2.54mm_Vertical, B.Cu at (332.7, 101.6)
- added FRAM_HEADER1: FRAM_Breakout_i2c_01x08, Connector_PinSocket_2.54mm:PinSocket_1x08_P2.54mm_Vertical, B.Cu at (381.0, 38.1)
- added J15: i2c encoder, Connector_PinSocket_2.54mm:PinSocket_1x05_P2.54mm_Vertical, F.Cu at (184.8, 77.5)
- added J16: i2c encoder, Connector_PinSocket_2.54mm:PinSocket_1x05_P2.54mm_Vertical, F.Cu at (161.9, 77.5)
- added J17: i2c encoder, Connector_PinSocket_2.54mm:PinSocket_1x05_P2.54mm_Vertical, F.Cu at (168.3, 94.0)
- added J18: i2c_header_2, Connector_PinSocket_2.54mm:PinSocket_1x04_P2.54mm_Vertical, B.Cu at (251.5, 124.5)
- added J18: i2c_header_2, Connector_PinSocket_2.54mm:PinSocket_1x04_P2.54mm_Vertical, B.Cu at (154.9, 124.5)
- added J19: i2c_header_2, Connector_PinSocket_2.54mm:PinSocket_1x04_P2.54mm_Vertical, F.Cu at (332.7, 124.5)
- added J19: i2c_header_2, Connector_PinSocket_2.54mm:PinSocket_1x04_P2.54mm_Vertical, F.Cu at (246.4, 124.5)
- added J20: Conn_01x11_Female, Connector_PinSocket_2.54mm:PinSocket_1x11_P2.54mm_Vertical, F.Cu at (304.8, 96.5)
- added J21: Conn_01x11_Male, Connector_PinHeader_2.54mm:PinHeader_1x11_P2.54mm_Vertical, B.Cu at (289.6, 132.1)
- added J21: Conn_01x11_Male, Connector_PinHeader_2.54mm:PinHeader_1x11_P2.54mm_Vertical, F.Cu at (370.8, 132.1)
- added J21: Conn_01x11_Male, Connector_PinHeader_2.54mm:PinHeader_1x11_P2.54mm_Vertical, B.Cu at (213.4, 96.5)
- added OLED_HEADER1: SSD1306_i2c_Oled_Conn, Display:Adafruit_SSD1306, F.Cu at (163.8, 32.4)
- added R10: 4.7K, Resistor_THT:R_Axial_DIN0204_L3.6mm_D1.6mm_P7.62mm_Horizontal, F.Cu at (77.5, 170.8)
- added R11: 220R, Resistor_THT:R_Axial_DIN0204_L3.6mm_D1.6mm_P7.62mm_Horizontal, F.Cu at (125.1, 142.9)
- added R12: R, Resistor_THT:R_Axial_DIN0204_L3.6mm_D1.6mm_P7.62mm_Horizontal, F.Cu at (194.3, 57.1)
- added R13: 220k, Resistor_THT:R_Axial_DIN0204_L3.6mm_D1.6mm_P7.62mm_Horizontal, F.Cu at (125.8, 19.7)
- added R14: 10k, Resistor_THT:R_Axial_DIN0204_L3.6mm_D1.6mm_P7.62mm_Horizontal, F.Cu at (114.1, 36.0)
- added R15: 22, Resistor_THT:R_Axial_DIN0204_L3.6mm_D1.6mm_P7.62mm_Horizontal, F.Cu at (125.8, 22.8)
- added R16: 22, Resistor_THT:R_Axial_DIN0204_L3.6mm_D1.6mm_P7.62mm_Horizontal, F.Cu at (125.8, 26.0)
- added R9: 220R, Resistor_THT:R_Axial_DIN0204_L3.6mm_D1.6mm_P7.62mm_Horizontal, F.Cu at (126.4, 160.7)
- added SPI_HEADER1: Conn_01x06_Female, Connector_PinSocket_2.54mm:PinSocket_1x06_P2.54mm_Vertical, B.Cu at (370.8, 45.7)
- added SW2: SW_Push_Dual, Button_Switch_THT:Push_E-Switch_KS01Q01, F.Cu at (201.1, 51.1)
- added U1: 6N138, Package_DIP:DIP-8_W7.62mm_Socket, F.Cu at (118.1, 155.6)
- added U4: MOS6581_6582_8580SID, Package_DIP:DIP-28_W15.24mm_Socket, F.Cu at (256.5, 48.3)
- added i2c_header1: i2c_spare, Connector_PinSocket_2.54mm:PinSocket_1x04_P2.54mm_Vertical, B.Cu at (363.2, 45.7)
- C1, C2, C3: footprint Capacitor_THT:C_Axial_L5.1mm_D3.1mm_P7.50mm_Horizontal -> Capacitor_THT:C_Disc_D8.0mm_W2.5mm_P5.00mm
- J10: footprint footprints:thonkiconn_fuzzySi -> AudioJacks:Jack_3.5mm_QingPu_WQP-PJ366ST_Vertical
- J11: value Conn_01x06_Female -> MIDI IN Conn_01x03_Male; footprint Connector_PinHeader_2.54mm:PinHeader_1x06_P2.54mm_Vertical -> Connector_PinSocket_2.54mm:PinSocket_1x03_P2.54mm_Vertical
- J12: value SSD1306_i2c_Oled_Conn_01x04_Female -> i2c encoder; footprint Connector_PinHeader_2.54mm:PinHeader_1x04_P2.54mm_Vertical -> Connector_PinSocket_2.54mm:PinSocket_1x05_P2.54mm_Vertical
- J13: value FRAM_Breakout_i2c_01x08 -> Euro power; footprint Connector_PinHeader_2.54mm:PinHeader_1x08_P2.54mm_Vertical -> Connector_IDC:IDC-Header_2x08_P2.54mm_Latch_Vertical; moved to B.Cu
- R1, R2, R3, R4, R8: footprint Resistor_THT:R_Axial_DIN0309_L9.0mm_D3.2mm_P12.70mm_Horizontal -> Resistor_THT:R_Axial_DIN0204_L3.6mm_D1.6mm_P7.62mm_Horizontal
- R5, R6: value R -> 10k; footprint Resistor_THT:R_Axial_DIN0309_L9.0mm_D3.2mm_P12.70mm_Horizontal -> Resistor_THT:R_Axial_DIN0204_L3.6mm_D1.6mm_P7.62mm_Horizontal
- R7: value R -> 100k; footprint Resistor_THT:R_Axial_DIN0309_L9.0mm_D3.2mm_P12.70mm_Horizontal -> Resistor_THT:R_Axial_DIN0204_L3.6mm_D1.6mm_P7.62mm_Horizontal
- U3: value PIMORONI_24v_ADC_1_ADS1015IDGS -> TL072; footprint Package_SO:TSSOP-10_3x3mm_P0.5mm -> Package_DIP:DIP-8_W7.62mm_Socket
- Y1: footprint Crystal:Crystal_AT310_D3.0mm_L10.0mm_Horizontal -> Crystal:Crystal_HC18-U_Vertical
- moved U7 215.4 mm to (63.5, 165.7)
- moved J13 188.4 mm to (381.0, 124.5)
- moved C3 178.1 mm to (31.8, 173.4), turned to 180 degrees
- moved Y1 148.3 mm to (246.4, 83.8), turned to 90 degrees
- moved J11 133.4 mm to (132.6, 147.9)
- moved U3 131.6 mm to (102.9, 19.5)
- moved C1 131.4 mm to (52.7, 102.2)
- moved R3 129.4 mm to (89.5, 148.0), turned to 90 degrees
- moved U2 124.7 mm to (256.5, 58.4)
- moved R1 122.3 mm to (89.5, 135.9), turned to 90 degrees
- moved D6 121.2 mm to (85.1, 155.6), turned to 180 degrees
- moved C2 120.5 mm to (60.3, 97.2), turned to 180 degrees
- moved D5 112.2 mm to (77.5, 150.5)
- moved D2 111.5 mm to (85.1, 165.7), turned to 180 degrees
- moved D4 110.8 mm to (85.1, 160.7), turned to 180 degrees
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Connections:
- C3 pad 1: GND -> Net-(C3-Pad1)
- J11 pad 1: Net-(C3-Pad2) -> GND
- J11 pad 2: MIDI_TX -> Net-(J10-PadR)
- J11 pad 3: MIDI_RX -> Net-(D7-Pad2)
- J12 pad 1: 3.3v -> GND
- J12 pad 2: GND -> +5V
- J12 pad 3: i2c_SCL -> i2c_SDA
- J12 pad 4: i2c_SDA -> i2c_SCL
- J13 pad 1: Net-(J13-Pad1) -> Net-(D8-Pad1)
- J13 pad 2: Net-(J13-Pad2) -> Net-(D8-Pad1)
- J13 pad 3: Net-(J13-Pad3) -> GND
- J13 pad 4: i2c_SDA -> GND
- J13 pad 5: i2c_SCL -> GND
- J13 pad 6: Net-(J13-Pad6) -> GND
- J13 pad 8: +5V -> GND
- J14 pad 2: Net-(J14-Pad2) -> GND
- J14 pad 3: Net-(J14-Pad3) -> JACK_OUT
- R4 pad 2: GND -> Net-(C3-Pad1)
- R6 pad 2: Net-(R6-Pad2) -> Net-(R13-Pad1)
- R7 pad 1: Net-(J14-Pad3) -> Net-(C4-Pad2)
- R7 pad 2: Net-(R6-Pad2) -> GND
- U2 pad 14: MIDI_RX -> MIDI_ATMEGA_RX
- U2 pad 25: Net-(U2-Pad25) -> Gate_1_IN
- U2 pad 26: Net-(U2-Pad26) -> Gate_2_IN
- U2 pad 27: Net-(U2-Pad27) -> Gate_3_IN
- U2 pad 28: Net-(U2-Pad28) -> BUTTON_B
- U2 pad 9: GND -> Net-(C3-Pad1)
- U3 pad 2: Net-(U3-Pad2) -> Net-(R13-Pad1)
- U3 pad 3: GND -> Net-(C4-Pad2)
- U3 pad 4: INPUT_A -> Net-(U3-Pad4)
- U3 pad 5: INPUT_B -> Net-(C5-Pad2)
- U3 pad 6: INPUT_C -> JACK_OUT
- U3 pad 7: Net-(U3-Pad7) -> JACK_OUT
- U3 pad 8: +5V -> +12V
Other:
- board outline added: 311.1 x 128.9 mm

Commit message: slightly updated
Parts:
- moved C7 307.6 mm to (365.8, 116.8)
- moved C6 306.2 mm to (365.8, 102.9)
- moved C4 221.3 mm to (294.6, 120.7)
- moved U1 209.6 mm to (290.8, 36.8), turned to 0 degrees
- moved U3 190.6 mm to (283.2, 81.3), turned to 90 degrees
- moved U7 130.7 mm to (153.7, 71.1)
- moved OLED_HEADER1 34.7 mm to (181.6, 62.2), turned to 180 degrees
- moved FRAM_HEADER1 34.5 mm to (370.8, 71.1), turned to 180 degrees
- moved U4 10.2 mm to (246.4, 47.0)
Connections:
- J18 pad 1: (no net) -> i2c_SDA
- J18 pad 2: (no net) -> i2c_SCL
- J18 pad 3: (no net) -> GND
- J18 pad 4: (no net) -> +5V
- J19 pad 1: (no net) -> i2c_SDA
- J19 pad 2: (no net) -> i2c_SCL
- J19 pad 3: (no net) -> GND
- J19 pad 4: (no net) -> +5V
- J21 pad 1: (no net) -> JACK_OUT (x2)
- J21 pad 10: (no net) -> INPUT_F (x2)
- J21 pad 11: (no net) -> GND (x2)
- J21 pad 2: (no net) -> Gate_1_IN (x2)
- J21 pad 3: (no net) -> Gate_2_IN (x2)
- J21 pad 4: (no net) -> Gate_3_IN (x2)
- J21 pad 5: (no net) -> INPUT_A (x2)
- J21 pad 6: (no net) -> INPUT_B (x2)
- J21 pad 7: (no net) -> INPUT_C (x2)
- J21 pad 8: (no net) -> INPUT_D (x2)
- J21 pad 9: (no net) -> INPUT_E (x2)
